File: BlueSTM32/BlueSTM32.kicad_pcb (KiCad board)
At the start: 4 copper layers, 40 x 40 mm, 63 parts, among them J1 TC2030-NL, J2 522071233, J3 USB4500-03-1-A_REVA, U1 OPA340NA, U2 BQ24040DSQR, U4 REF2033, U5 LT1304CS8-3.3-PBF, U6 LSM6DSRTR, U7 W25N02KVZEIR TR, U8 STM32WB55RGVx, X2 32.768kHz, X4 32MHz

Commit message: Final ordered version of the board with gerbers
Parts:
- moved R9 0.42 mm to (167.1, 108.3)
Routing:
- net /Microcontroller/SWD_RST: track 22.7 -> 24.8 mm
- net /Microcontroller/LSE_X2_out: track 7.42 -> 8.45 mm
- net /Microcontroller/Flash_DI(IO0): track 12.6 -> 13.6 mm
- net /Microcontroller/BOOT0: track 7.78 -> 8.73 mm, vias 0 -> 2
- net USB_D-: track 13.9 -> 13.0 mm
- net Net-(U2-~{PG}): track 8.21 -> 9.07 mm
- net GND: track 121.1 -> 121.8 mm
- net USB_D+: track 14.2 -> 13.6 mm

Commit message: Final Version of the board
Parts:
- added C13: 4.7uF, Capacitor_SMD:C_0402_1005Metric_Pad0.74x0.62mm_HandSolder, F.Cu at (180.8, 118.8)
- added L2: 10u, Inductor_SMD:L_0805_2012Metric_Pad1.15x1.40mm_HandSolder, F.Cu at (188.3, 121.6)
- renumbered CHG to D1, PG to D2, BAT+ to TP1, GND to TP2, X4 to X1
Connections:
- C7 pad 2: Net-(U1-+) -> Net-(U1--)
- C8 pad 1: Net-(U1-+) -> Net-(U1--)
- L1 pad 2: Net-(D3-A) -> Net-(U5-SW)
- R3 pad 1: Net-(U1-+) -> Net-(U1--)
- U1 pad 3: Net-(U1-+) -> Piezoelectric_-
- U1 pad 4: Piezoelectric_- -> Net-(U1--)
- U5 pad 4: Net-(D3-A) -> Net-(U5-SW)
Routing:
- net Net-(U1--): track 0.00 -> 13.0 mm, vias 0 -> 2
- net Net-(U1-+): track 6.95 -> 0.00 mm
- net Net-(U5-SW): track 0.00 -> 5.51 mm
- net Net-(D3-A): track 5.95 -> 7.89 mm
- net GND: track 121.8 -> 123.5 mm
