File: BlueSTM32/Microcontroller.kicad_sch (KiCad schematic)
At the start: 19 parts, among them J1 TC2030-NL, U7 W25N02KVZEIR TR, U8 STM32WB55RGVx, X3 32.768kHz, X4 32MHz

Commit message: Better Final Layout
Parts:
- renumbered X4 to X1, X3 to X2
Changed lines of the file:
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@@
 		(on_board yes)
 		(dnp no)
-		(property "Reference" "X4"
+		(property "Reference" "X1"
 			(at 168.91 130.81 0)
 			(effects
@@
 			(project "BlueSTM32"
 				(path "/0813bd8c-34b7-4d98-8a6f-d3ea444f1dbc/d60c4563-988a-402c-8446-26bba05170b9"
-					(reference "X4")
+					(reference "X1")
 					(unit 1)
 				)
@@
 		(dnp no)
 		(fields_autoplaced yes)
-		(property "Reference" "X3"
+		(property "Reference" "X2"
 			(at 144.78 149.86 0)
 			(effects
@@
 			(project "BlueSTM32"
 				(path "/0813bd8c-34b7-4d98-8a6f-d3ea444f1dbc/d60c4563-988a-402c-8446-26bba05170b9"
-					(reference "X3")
-					(unit 1)
-				)
+					(reference "X2")
+					(unit 1)
+				)
